Commit message: Fixed color problems

File: my_robot/urdf/my_robot.xacro (robot description, xacro)
@@ -2,13 +2,4 @@
 <robot name="my_robot" xmlns:xacro="http://www.ros.org/wiki/xacro">
 <xacro:include filename="$(find my_robot)/urdf/my_robot.gazebo" />
-  <material name="chasis_color">
-   <color rgba="0 0.8 0.8 1"/>
-  </material>
-  <material name="camera_color">
-   <color rgba="0.8 0.3 0.3 1"/>
-  </material>
-  <material name="wheel_color">
-   <color rgba="0.8 0.3 0.3 1"/>
-  </material>
   <link name="robot_footprint"></link>
   <joint name="robot_footprint_joint" type="fixed">
@@ -39,28 +30,27 @@
         <box size=".6 .2 .1"/>
       </geometry>
-      <material name="chasis_color"/>
     </visual>
     <collision name='back_caster_collision'>
-      <origin xyz="-0.15 0 -0.05" rpy=" 0 0 0"/>
+      <origin xyz="-0.15 0 -0.1" rpy=" 0 0 0"/>
       <geometry>
-        <sphere radius="0.0499"/>
+        <sphere radius="0.1"/>
       </geometry>
     </collision>
     <visual name='back_caster_visual'>
-      <origin xyz="-0.15 0 -0.05" rpy=" 0 0 0"/>
+      <origin xyz="-0.15 0 -0.1" rpy=" 0 0 0"/>
       <geometry>
-        <sphere radius="0.05"/>
+        <sphere radius="0.1"/>
       </geometry>
     </visual>
     <collision name='front_caster_collision'>
-      <origin xyz="0.15 0 -0.05" rpy=" 0 0 0"/>
+      <origin xyz="0.15 0 -0.1" rpy=" 0 0 0"/>
       <geometry>
-        <sphere radius="0.0499"/>
+        <sphere radius="0.1"/>
       </geometry>
     </collision>
     <visual name='front_caster_visual'>
-      <origin xyz="0.15 0 -0.05" rpy=" 0 0 0"/>
+      <origin xyz="0.15 0 -0.1" rpy=" 0 0 0"/>
       <geometry>
-        <sphere radius="0.05"/>
+        <sphere radius="0.1"/>
       </geometry>
     </visual>
@@ -88,5 +78,4 @@
         <cylinder radius=".2" length="0.05"/>
       </geometry>
-      <material name="wheel_color"/>
     </visual>
    </link>
@@ -121,5 +110,4 @@
         <cylinder radius=".2" length="0.05"/>
       </geometry>
-      <material name="wheel_color"/>
     </visual>
    </link>
@@ -154,14 +142,13 @@
         <box size=".05 .05 .05"/>
       </geometry>
-    <material name="camera_color"/>
     </visual>
    </link>
    <joint type="fixed" name="camera_joint">
-     <origin xyz="0.2 0 0" rpy="0 0 0"/>
+     <origin xyz="0.3 0 0" rpy="0 0 0"/>
      <child link="camera"/>
      <parent link="chassis"/>
      <axis xyz="0 1 0" rpy="0 0 0"/>
    </joint>
-<link name='hokuyo'>
+   <link name='hokuyo'>
     <pose>0 0 0 0 0 0</pose>
     <inertial>
@@ -193,3 +180,18 @@
      <axis xyz="0 1 0" rpy="0 0 0"/>
    </joint>
+   <gazebo reference="chassis">
+    <material>Gazebo/Green</material>
+    </gazebo>
+    <gazebo reference="left_wheel">
+    <material>Gazebo/Black</material>
+    </gazebo>
+    <gazebo reference="right_wheel">
+    <material>Gazebo/Black</material>
+    </gazebo>
+    <gazebo reference="chassis">
+    <material>Gazebo/Green</material>
+    </gazebo>
+    <gazebo reference="camera">
+    <material>Gazebo/Yellow</material>
+    </gazebo>
 </robot>
